Commit message: chore: update world file and add launch file
need more feature in world for camera capturing

File: my_robot/urdf/my_robot.xacro (robot description, xacro)
@@ -113,5 +113,5 @@
 </link>
 <joint name="camera_optical_joint" type="fixed">
-    <origin xyz="0 0 0" rpy="-1.5707 0 -1.5707"/>
+    <origin xyz="0 0 0" rpy="-1.57 0 -1.57"/>
     <!-- camera link -->
     <parent link="camera"/>
